Commit message: add tpm_moveit
* add package: tpm_moveit
* rm package: tpm_demo
  (move launch file to tpm_moveit & tpm_core_node)

File: tpm_description/urdf/ar3_no_col.urdf.xacro (robot description, xacro)
@@ -11,10 +11,4 @@
         <material name="orange"/>
       </visual>
-      <collision>
-        <origin xyz="0 0 0" rpy="0 0 0" />
-        <geometry>
-          <mesh filename="package://tpm_description/meshes/ar3/base_link.stl" />
-        </geometry>
-      </collision>
     </link>
     <joint name="joint1" type="revolute">
@@ -33,16 +27,4 @@
         <material name="blue"/>
       </visual>
-      <collision>
-        <origin xyz="0 0 0" rpy="0 0 0" />
-        <geometry>
-          <mesh filename="package://tpm_description/meshes/ar3/link_1.stl" />
-        </geometry>
-      </collision>
-      <inertial>
-        <origin xyz="-0.022706 0.04294 -0.12205" rpy="0 0 0" />
-        <mass value="0.88065" />
-        <inertia ixx="0.0034" ixy="0.00042296" ixz="-0.00089231"
-                 iyy="0.0041778" iyz="0.0010848" izz="0.0027077" />
-      </inertial>
     </link>
     <joint name="joint2" type="revolute">
@@ -63,10 +45,4 @@
         <material name="green"/>
       </visual>
-      <collision>
-        <origin xyz="0 0 0" rpy="0 0 0" />
-        <geometry>
-          <mesh filename="package://tpm_description/meshes/ar3/link_2.stl" />
-        </geometry>
-      </collision>
     </link>
     <joint name="joint3" type="revolute">
@@ -87,10 +63,4 @@
         <material name="red"/>
       </visual>
-      <collision>
-        <origin xyz="0 0 0" rpy="0 0 0" />
-        <geometry>
-          <mesh filename="package://tpm_description/meshes/ar3/link_3.stl" />
-        </geometry>
-      </collision>
     </link>
     <joint name="joint4" type="revolute">
@@ -109,10 +79,4 @@
         <material name="blue"/>
       </visual>
-      <collision>
-        <origin xyz="0 0 0" rpy="0 0 0" />
-        <geometry>
-          <mesh filename="package://tpm_description/meshes/ar3/link_4.stl" />
-        </geometry>
-      </collision>
     </link>
     <joint name="joint5" type="revolute">
@@ -131,10 +95,4 @@
         <material name="green"/>
       </visual>
-      <collision>
-        <origin xyz="0 0 0" rpy="0 0 0" />
-        <geometry>
-          <mesh filename="package://tpm_description/meshes/ar3/link_5.stl" />
-        </geometry>
-      </collision>
     </link>
     <joint name="joint6" type="revolute">
@@ -153,10 +111,4 @@
         <material name="orange"/>
       </visual>
-      <collision>
-        <origin xyz="0 0 0" rpy="0 0 0" />
-        <geometry>
-          <mesh filename="package://tpm_description/meshes/ar3/link_6.stl" />
-        </geometry>
-      </collision>
     </link>
 </robot>
